File: Underside.kicad_sch (KiCad schematic)
At the start: 5 parts, among them J1 AE-MICRO-SD-DIP, U1 DPS310, U2 URM-37, U3 SeeeduinoXIAO

Commit message: update to 24th, add UART pullup
Parts:
- added JP1: SolderJumper_2_Open, symbol Jumper:SolderJumper_2_Open
- added R1: 1k, symbol Device:R
Connections:
- net +3.3V: now also JP1.2 (B)
- net DTXR: now also R1.2
- new net: JP1.1 (A), R1.1
- no-connect marks 0 -> 16
Other:
- company: (none) -> TORICA-24th
- title: (none) -> Underside
- moved on the sheet: J1, U1, U2, U3

Commit message: Update PCB_Under
Parts:
- JP1: footprint (none) -> Jumper:SolderJumper-2_P1.3mm_Open_RoundedPad1.0x1.5mm
- R1: footprint (none) -> Resistor_THT:R_Axial_DIN0204_L3.6mm_D1.6mm_P7.62mm_Horizontal
Changed lines of the file:
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@@
       (effects (font (size 1.27 1.27)) (justify left))
     )
-    (property "Footprint" "" (at 33.782 104.775 90)
+    (property "Footprint" "Resistor_THT:R_Axial_DIN0204_L3.6mm_D1.6mm_P7.62mm_Horizontal" (at 33.782 104.775 90)
       (effects (font (size 1.27 1.27)) hide)
     )
@@
       (effects (font (size 1.27 1.27)) (justify right))
     )
-    (property "Footprint" "" (at 35.56 92.71 0)
+    (property "Footprint" "Jumper:SolderJumper-2_P1.3mm_Open_RoundedPad1.0x1.5mm" (at 35.56 92.71 0)
       (effects (font (size 1.27 1.27)) hide)
     )
